Commit message: cambios rviz y joint gui

File: proyecto/urdf/proyecto.urdf (robot description, URDF)
Before this commit: robot proyecto, 6 links, 5 joints
Links:
- removed link dummy
- added link odom
Joints:
- joint dummy_joint: parent dummy -> odom
- joint motor_1: axis 0 1 0 -> 0 0 1
- joint motor_2: axis 0 1 0 -> 0 0 1
- joint motor_3: axis 0 1 0 -> 0 0 1
- joint motor_4: axis 0 1 0 -> 0 0 1

Commit message: Agregar archivos fuente

File: proyecto/urdf/proyecto.urdf (robot description, URDF)
Before this commit: robot proyecto, 5 links, 4 joints
Links:
- added link dummy
Joints:
- added joint dummy_joint: type fixed, parent dummy, child base_link
- joint motor_1: axis 0 0 0 -> 0 1 0
- joint motor_2: axis 0 0 0 -> 0 1 0
- joint motor_3: axis 0 0 0 -> 0 1 0
- joint motor_4: axis 0 0 0 -> 0 1 0

Commit message: creacion xacro

File: proyecto/urdf/proyecto.urdf (robot description, URDF)
Before this commit: robot proyecto, 6 links, 5 joints
Links:
- link rueda_2: mass 1.16170802075831 -> 1.1617081622077; geometry collision mesh filename=package://proyecto/meshes/rueda_1.STL; visual mesh filename=package://proyecto/meshes/rueda_1.STL
- link rueda_3: mass 1.16170796588524 -> 1.1617081622077; geometry collision mesh filename=package://proyecto/meshes/rueda_1.STL; visual mesh filename=package://proyecto/meshes/rueda_1.STL
- link rueda_4: mass 1.16170814603751 -> 1.1617081622077; geometry collision mesh filename=package://proyecto/meshes/rueda_1.STL; visual mesh filename=package://proyecto/meshes/rueda_1.STL
Joints:
- joint motor_1: origin xyz=-0.206 -0.13662 -0.041 rpy=1.5708 0 0 -> xyz=-0.206 -0.13662 -0.041 rpy=1.5707963267948966 0 0
- joint motor_2: origin xyz=0.206 -0.13722 -0.041 rpy=1.5708 0 0 -> xyz=-0.206 -0.13662 -0.041 rpy=1.5707963267948966 0 0
- joint motor_3: origin xyz=0.206 0.40485 -0.041 rpy=1.5708 0 0 -> xyz=-0.206 -0.13662 -0.041 rpy=1.5707963267948966 0 0
- joint motor_4: origin xyz=-0.206 0.40485 -0.041 rpy=1.5708 0 0 -> xyz=-0.206 -0.13662 -0.041 rpy=1.5707963267948966 0 0

Commit message: add urdf

File: proyecto/urdf/proyecto.urdf (robot description, URDF)
Before this commit: robot proyecto, 6 links, 5 joints
Links:
- removed link odom
- added link dummy
- link rueda_2: mass 1.1617081622077 -> 1.16170802075831
- link rueda_3: mass 1.1617081622077 -> 1.16170796588524
- link rueda_4: mass 1.1617081622077 -> 1.16170814603751
Joints:
- joint dummy_joint: parent odom -> dummy
- joint motor_1: axis 0 0 1 -> 0 1 0; origin xyz=-0.206 -0.13662 -0.041 rpy=1.5707963267948966 0 0 -> xyz=-0.206 -0.13662 -0.041 rpy=1.5708 0 0
- joint motor_2: axis 0 0 1 -> 0 1 0; origin xyz=-0.206 -0.13662 -0.041 rpy=1.5707963267948966 0 0 -> xyz=0.206 -0.13722 -0.041 rpy=1.5708 0 0
- joint motor_3: axis 0 0 1 -> 0 1 0; origin xyz=-0.206 -0.13662 -0.041 rpy=1.5707963267948966 0 0 -> xyz=0.206 0.40485 -0.041 rpy=1.5708 0 0
- joint motor_4: axis 0 0 1 -> 0 1 0; origin xyz=-0.206 -0.13662 -0.041 rpy=1.5707963267948966 0 0 -> xyz=-0.206 0.40485 -0.041 rpy=1.5708 0 0

File: proyecto/urdf/proyecto.urdf.xacro (robot description, xacro)
@@ -5,6 +5,6 @@
   <xacro:property name="back_wheel_y" value="0.40485" />
   <xacro:property name="wheel_z" value="-0.041" />
-  <xacro:property name="wheel_radius" value="78.5" />
-  <xacro:property name="wheel_width" value="15.8" />
+  <xacro:property name="wheel_radius" value="0.0785" />
+  <xacro:property name="wheel_width" value="0.0158" />
   <xacro:property name="chasis_lenght" value="58.1"/>
   <xacro:property name="chasis_width" value="52.9"/>
@@ -13,4 +13,10 @@
   <xacro:macro name="wheel" params="suffix *joint_pose">
     <link name="rueda_${suffix}">
+        <inertial>
+          <origin xyz="-5.707782267661E-07 1.62246123321108E-07 -0.0158002809636204" rpy="0 0 0"/>
+          <mass value="1.1617081622077"/>
+          <inertia ixx="0.00236389228715147" ixy="4.31489359287888E-09" ixz="-1.0352494720813E-08"
+                  iyy="0.00236389275249923" iyz="-3.84382849696802E-10" izz="0.00380474886030968"/>
+        </inertial>
       <visual>
         <origin xyz="0 0 0" rpy="0 0 0"/>
@@ -25,13 +31,8 @@
         <origin xyz="0 0 0" rpy="0 0 0"/>
           <geometry>
-            <cylinder radius="${wheel_radius}" length="${wheel_width}"/>
+             <cylinder radius="${wheel_radius}" length="${wheel_width}"/>
+            <!-- <mesh filename="package://proyecto/meshes/rueda_1.STL"/>-->
           </geometry>
       </collision>
-        <inertial>
-          <origin xyz="-5.707782267661E-07 1.62246123321108E-07 -0.0158002809636204" rpy="0 0 0"/>
-          <mass value="1.1617081622077"/>
-          <inertia ixx="0.00236389228715147" ixy="4.31489359287888E-09" ixz="-1.0352494720813E-08"
-                  iyy="0.00236389275249923" iyz="-3.84382849696802E-10" izz="0.00380474886030968"/>
-        </inertial>
     </link>
     <joint name="motor_${suffix}" type="continuous">
@@ -84,5 +85,5 @@
       <origin xyz="0 0 0" rpy="0 0 0"/>
       <geometry>
-              <box size="${chasis_lenght} ${chasis_width} ${chasis_height}"/>
+              <mesh filename="package://proyecto/meshes/base_link.STL"/>
       </geometry>
     </collision>
