Commit message: rviz con xacro

File: proyecto/urdf/proyecto.urdf.xacro (robot description, xacro)
@@ -1,106 +1,76 @@
 <?xml version="1.0" encoding="utf-8"?>
-<!-- This URDF was automatically created by SolidWorks to URDF Exporter! Originally created by Stephen Brawner (brawner@gmail.com)
-     Commit Version: 1.6.0-4-g7f85cfe  Build Version: 1.6.7995.38578
-     For more information, please see http://wiki.ros.org/sw_urdf_exporter -->
 <robot name="proyecto" xmlns:xacro="http://www.ros.org/wiki/xacro">
-  <!-- <xacro:property name="wheel_mass" value="1.1617081622077"/>  Asi declaro constantes -->
-  <xacro:property name="pi" value="3.141592653589793" />
   <xacro:macro name="wheel" params="suffix">
-  <link name = "rueda_${suffix}">
+    <link name="rueda_${suffix}">
+      <inertial>
+        <origin xyz="-5.707782267661E-07 1.62246123321108E-07 -0.0158002809636204" rpy="0 0 0"/>
+        <mass value="1.1617081622077"/>
+        <inertia ixx="0.00236389228715147" ixy="4.31489359287888E-09" ixz="-1.0352494720813E-08"
+                 iyy="0.00236389275249923" iyz="-3.84382849696802E-10" izz="0.00380474886030968"/>
+      </inertial>
+      <visual>
+        <origin xyz="0 0 0" rpy="0 0 0"/>
+        <geometry>
+          <mesh filename="package://proyecto/meshes/rueda_${suffix}.STL"/>
+        </geometry>
+        <material name="">
+          <color rgba="0.792156862745098 0.819607843137255 0.933333333333333 1"/>
+        </material>
+      </visual>
+      <collision>
+        <origin xyz="0 0 0" rpy="0 0 0"/>
+        <geometry>
+          <mesh filename="package://proyecto/meshes/rueda_${suffix}.STL"/>
+        </geometry>
+      </collision>
+    </link>
+    <joint name="motor_${suffix}" type="continuous">
+      <origin xyz="-0.206 -0.13662 -0.041" rpy="${pi/2.0} 0 0"/>
+      <parent link="base_link"/>
+      <child link="rueda_${suffix}"/>
+      <axis xyz="0 0 1"/>
+    </joint>
+    <transmission name="tran_${suffix}">
+      <type>transmission_interface/SimpleTransmission</type>
+      <joint name="motor_${suffix}">
+        <hardwareInterface>hardware_interface/VelocityJointInterface</hardwareInterface>
+      </joint>
+      <actuator name="motor_${suffix}">
+        <hardwareInterface>hardware_interface/VelocityJointInterface</hardwareInterface>
+        <mechanicalReduction>1</mechanicalReduction>
+      </actuator>
+    </transmission>
+  </xacro:macro>
+  <xacro:wheel suffix="1"/>
+  <xacro:wheel suffix="2"/>
+  <xacro:wheel suffix="3"/>
+  <xacro:wheel suffix="4"/>
+  <link name="odom"/>
+  <link name="base_link">
     <inertial>
-      <origin
-        xyz="-5.707782267661E-07 1.62246123321108E-07 -0.0158002809636204"
-        rpy="0 0 0" />
-      <mass
-        value="1.1617081622077" />
-      <inertia
-        ixx="0.00236389228715147" ixy="4.31489359287888E-09" ixz="-1.0352494720813E-08"
-        iyy="0.00236389275249923" iyz="-3.84382849696802E-10" izz="0.00380474886030968" />
+      <origin xyz="0.0238551640441538 0.0295955080939407 -0.150383488449588" rpy="0 0 0"/>
+      <mass value="4.58423641056187"/>
+      <inertia ixx="0.0171426025781744" ixy="-0.00117297644050985" ixz="-6.44110873168587E-07"
+               iyy="0.0611975209416774" iyz="-1.44180477906026E-08" izz="0.047936942239142"/>
     </inertial>
     <visual>
-      <origin
-        xyz="0 0 0" rpy="0 0 0" />
+      <origin xyz="0 0 0" rpy="0 0 0"/>
       <geometry>
-        <mesh
-          filename="package://proyecto/meshes/rueda_1.STL" />
+        <mesh filename="package://proyecto/meshes/base_link.STL"/>
       </geometry>
-      <material
-        name="">
-        <color
-          rgba="0.792156862745098 0.819607843137255 0.933333333333333 1" />
+      <material name="">
+        <color rgba="0.996078431372549 0.996078431372549 1 1"/>
       </material>
     </visual>
     <collision>
-      <origin
-        xyz="0 0 0" rpy="0 0 0" />
+      <origin xyz="0 0 0" rpy="0 0 0"/>
       <geometry>
-        <mesh
-          filename="package://proyecto/meshes/rueda_1.STL" />
+        <mesh filename="package://proyecto/meshes/base_link.STL"/>
       </geometry>
     </collision>
   </link>
-  <joint name="motor_${suffix}" type="continuous">
-    <origin
-      xyz="-0.206 -0.13662 -0.041"
-      rpy="${pi/2.0} 0 0" />
-    <parent
-      link="base_link" />
-    <child
-      link="rueda_${suffix}" />
-    <axis xyz="0 0 1" />
-  </joint>
-    <transmission name="tran_${suffix}">
-    <type>transmission_interface/SimpleTransmission</type>
-    <joint name="motor_${suffix}">
-      <hardwareInterface>hardware_interface/VelocityJointInterface</hardwareInterface>
-    </joint>
-    <actuator name="motor_${suffix}">
-      <hardwareInterface>hardware_interface/VelocityJointInterface</hardwareInterface>
-      <mechanicalReduction>1</mechanicalReduction>
-    </actuator>
-  </transmission>
-  </xacro:macro>
-  <xacro:wheel suffix="1"> </xacro:wheel>
-  <xacro:wheel suffix="2"> </xacro:wheel>
-  <xacro:wheel suffix="3"> </xacro:wheel>
-  <xacro:wheel suffix="4"> </xacro:wheel>
-  <link name="odom">
- </link>
-  <link
-    name="base_link">
-    <inertial>
-      <origin
-        xyz="0.0238551640441538 0.0295955080939407 -0.150383488449588" rpy="0 0 0" />
-      <mass
-        value="4.58423641056187" />
-      <inertia
-        ixx="0.0171426025781744" ixy="-0.00117297644050985" ixz="-6.44110873168587E-07"
-        iyy="0.0611975209416774" iyz="-1.44180477906026E-08" izz="0.047936942239142" />
-    </inertial>
-    <visual>
-      <origin
-        xyz="0 0 0" rpy="0 0 0" />
-      <geometry>
-        <mesh
-          filename="package://proyecto/meshes/base_link.STL" />
-      </geometry>
-      <material
-        name="">
-        <color
-          rgba="0.996078431372549 0.996078431372549 1 1" />
-      </material>
-    </visual>
-    <collision>
-      <origin
-        xyz="0 0 0" rpy="0 0 0" />
-      <geometry>
-        <mesh
-          filename="package://proyecto/meshes/base_link.STL" />
-      </geometry>
-    </collision>
-  </link>
-    <joint name="dummy_joint" type="fixed">
+  <joint name="dummy_joint" type="fixed">
     <parent link="odom"/>
-     <child link="base_link"/>
+    <child link="base_link"/>
   </joint>
 </robot>

Commit message: correction in xacro and gazebo spawn

File: proyecto/urdf/proyecto.urdf.xacro (robot description, xacro)
@@ -1,5 +1,9 @@
 <?xml version="1.0" encoding="utf-8"?>
 <robot name="proyecto" xmlns:xacro="http://www.ros.org/wiki/xacro">
-  <xacro:macro name="wheel" params="suffix">
+  <xacro:property name="wheel_x" value="0.206" />
+  <xacro:property name="front_wheel_y" value="-0.13662" />
+  <xacro:property name="back_wheel_y" value="0.40485" />
+  <xacro:property name="wheel_z" value="-0.041" />
+  <xacro:macro name="wheel" params="suffix *joint_pose">
     <link name="rueda_${suffix}">
       <inertial>
@@ -8,25 +12,25 @@
         <inertia ixx="0.00236389228715147" ixy="4.31489359287888E-09" ixz="-1.0352494720813E-08"
                  iyy="0.00236389275249923" iyz="-3.84382849696802E-10" izz="0.00380474886030968"/>
-      </inertial>
+        </inertial>
       <visual>
         <origin xyz="0 0 0" rpy="0 0 0"/>
-        <geometry>
-          <mesh filename="package://proyecto/meshes/rueda_${suffix}.STL"/>
-        </geometry>
-        <material name="">
-          <color rgba="0.792156862745098 0.819607843137255 0.933333333333333 1"/>
-        </material>
+          <geometry>
+            <mesh filename="package://proyecto/meshes/rueda_1.STL"/>
+          </geometry>
+          <material name="">
+            <color rgba="0.792156862745098 0.819607843137255 0.933333333333333 1"/>
+          </material>
       </visual>
       <collision>
         <origin xyz="0 0 0" rpy="0 0 0"/>
-        <geometry>
-          <mesh filename="package://proyecto/meshes/rueda_${suffix}.STL"/>
-        </geometry>
+          <geometry>
+            <mesh filename="package://proyecto/meshes/rueda_1.STL"/>
+          </geometry>
       </collision>
     </link>
     <joint name="motor_${suffix}" type="continuous">
-      <origin xyz="-0.206 -0.13662 -0.041" rpy="${pi/2.0} 0 0"/>
       <parent link="base_link"/>
       <child link="rueda_${suffix}"/>
+      <xacro:insert_block name="joint_pose" />
       <axis xyz="0 0 1"/>
     </joint>
@@ -36,5 +40,5 @@
         <hardwareInterface>hardware_interface/VelocityJointInterface</hardwareInterface>
       </joint>
-      <actuator name="motor_${suffix}">
+      <actuator name="motor${suffix}">
         <hardwareInterface>hardware_interface/VelocityJointInterface</hardwareInterface>
         <mechanicalReduction>1</mechanicalReduction>
@@ -42,8 +46,16 @@
     </transmission>
   </xacro:macro>
-  <xacro:wheel suffix="1"/>
-  <xacro:wheel suffix="2"/>
-  <xacro:wheel suffix="3"/>
-  <xacro:wheel suffix="4"/>
+  <xacro:wheel suffix="1">
+    <origin xyz="${-wheel_x} ${front_wheel_y} ${wheel_z}" rpy="${pi/2} 0 0" />
+  </xacro:wheel>
+  <xacro:wheel suffix="2">
+    <origin xyz="${wheel_x} ${front_wheel_y} ${wheel_z}" rpy="${pi/2} 0 0" />
+  </xacro:wheel>
+  <xacro:wheel suffix="3">
+    <origin xyz="${wheel_x} ${back_wheel_y} ${wheel_z}" rpy="${pi/2} 0 0" />
+  </xacro:wheel>
+  <xacro:wheel suffix="4">
+    <origin xyz="${-wheel_x} ${back_wheel_y} ${wheel_z}" rpy="${pi/2} 0 0" />
+  </xacro:wheel>
   <link name="odom"/>
   <link name="base_link">

Commit message: change to controller and xacro

File: proyecto/urdf/proyecto.urdf.xacro (robot description, xacro)
@@ -5,4 +5,6 @@
   <xacro:property name="back_wheel_y" value="0.40485" />
   <xacro:property name="wheel_z" value="-0.041" />
+  <xacro:property name="wheel_radius" value="78.5" />
+  <xacro:property name="wheel_width" value="158" />
   <xacro:macro name="wheel" params="suffix *joint_pose">
     <link name="rueda_${suffix}">
@@ -25,5 +27,5 @@
         <origin xyz="0 0 0" rpy="0 0 0"/>
           <geometry>
-            <mesh filename="package://proyecto/meshes/rueda_1.STL"/>
+            <cylinder radius="${wheel_radius}" length="${wheel_width}"/>
           </geometry>
       </collision>
@@ -61,5 +63,5 @@
   <link name="base_link">
     <inertial>
-      <origin xyz="0.0238551640441538 0.0295955080939407 -0.150383488449588" rpy="0 0 0"/>
+      <origin xyz="0.0238551640441538 0.0295955080939407 0" rpy="0 0 0"/>
       <mass value="4.58423641056187"/>
       <inertia ixx="0.0171426025781744" ixy="-0.00117297644050985" ixz="-6.44110873168587E-07"
@@ -86,3 +88,7 @@
     <child link="base_link"/>
   </joint>
+ <gazebo>
+    <plugin name="gazebo_ros_control" filename="libgazebo_ros_control.so">
+    </plugin>
+  </gazebo>
 </robot>

Commit message: test

File: proyecto/urdf/proyecto.urdf.xacro (robot description, xacro)
@@ -6,13 +6,11 @@
   <xacro:property name="wheel_z" value="-0.041" />
   <xacro:property name="wheel_radius" value="78.5" />
-  <xacro:property name="wheel_width" value="158" />
+  <xacro:property name="wheel_width" value="15.8" />
+  <xacro:property name="chasis_lenght" value="58.1"/>
+  <xacro:property name="chasis_width" value="52.9"/>
+  <xacro:property name="chasis_height" value="25.3"/>
+  <xacro:property name="pi" value="3.14159265358979323846" />
   <xacro:macro name="wheel" params="suffix *joint_pose">
     <link name="rueda_${suffix}">
-      <inertial>
-        <origin xyz="-5.707782267661E-07 1.62246123321108E-07 -0.0158002809636204" rpy="0 0 0"/>
-        <mass value="1.1617081622077"/>
-        <inertia ixx="0.00236389228715147" ixy="4.31489359287888E-09" ixz="-1.0352494720813E-08"
-                 iyy="0.00236389275249923" iyz="-3.84382849696802E-10" izz="0.00380474886030968"/>
-        </inertial>
       <visual>
         <origin xyz="0 0 0" rpy="0 0 0"/>
@@ -30,4 +28,10 @@
           </geometry>
       </collision>
+        <inertial>
+          <origin xyz="-5.707782267661E-07 1.62246123321108E-07 -0.0158002809636204" rpy="0 0 0"/>
+          <mass value="1.1617081622077"/>
+          <inertia ixx="0.00236389228715147" ixy="4.31489359287888E-09" ixz="-1.0352494720813E-08"
+                  iyy="0.00236389275249923" iyz="-3.84382849696802E-10" izz="0.00380474886030968"/>
+        </inertial>
     </link>
     <joint name="motor_${suffix}" type="continuous">
@@ -42,5 +46,5 @@
         <hardwareInterface>hardware_interface/VelocityJointInterface</hardwareInterface>
       </joint>
-      <actuator name="motor${suffix}">
+      <actuator name="actuator_${suffix}">
         <hardwareInterface>hardware_interface/VelocityJointInterface</hardwareInterface>
         <mechanicalReduction>1</mechanicalReduction>
@@ -80,5 +84,5 @@
       <origin xyz="0 0 0" rpy="0 0 0"/>
       <geometry>
-        <mesh filename="package://proyecto/meshes/base_link.STL"/>
+              <box size="${chasis_lenght} ${chasis_width} ${chasis_height}"/>
       </geometry>
     </collision>

Commit message: xacro changes

File: proyecto/urdf/proyecto.urdf.xacro (robot description, xacro)
@@ -67,5 +67,5 @@
   <link name="base_link">
     <inertial>
-      <origin xyz="0.0238551640441538 0.0295955080939407 0" rpy="0 0 0"/>
+      <origin xyz="0.0238551640441538 0.0295955080939407 -0.150383488449588" rpy="0 0 0"/>
       <mass value="4.58423641056187"/>
       <inertia ixx="0.0171426025781744" ixy="-0.00117297644050985" ixz="-6.44110873168587E-07"

Commit message: creation of a workink controller, now gazebo works

File: proyecto/urdf/proyecto.urdf.xacro (robot description, xacro)
@@ -6,9 +6,13 @@
   <xacro:property name="wheel_z" value="-0.041" />
   <xacro:property name="wheel_radius" value="0.0785" />
-  <xacro:property name="wheel_width" value="0.0158" />
-  <xacro:property name="chasis_lenght" value="58.1"/>
-  <xacro:property name="chasis_width" value="52.9"/>
-  <xacro:property name="chasis_height" value="25.3"/>
+  <xacro:property name="wheel_width" value="0.078" />
+  <xacro:property name="chasis_lenght" value="0.581"/>
+  <xacro:property name="chasis_width" value="0.529"/>
+  <xacro:property name="chasis_height" value="0.253"/>
   <xacro:property name="pi" value="3.14159265358979323846" />
+  <material name="dark_grey"><color rgba="0.2 0.2 0.2 1.0" /></material>
+  <material name="light_grey"><color rgba="0.4 0.4 0.4 1.0" /></material>
+  <material name="yellow"><color rgba="0.8 0.8 0.0 1.0" /></material>
+  <material name="black"><color rgba="0.15 0.15 0.15 1.0" /></material>
   <xacro:macro name="wheel" params="suffix *joint_pose">
     <link name="rueda_${suffix}">
@@ -24,10 +28,8 @@
             <mesh filename="package://proyecto/meshes/rueda_1.STL"/>
           </geometry>
-          <material name="">
-            <color rgba="0.792156862745098 0.819607843137255 0.933333333333333 1"/>
-          </material>
+          <material name="black" />
       </visual>
       <collision>
-        <origin xyz="0 0 0" rpy="0 0 0"/>
+        <origin xyz="0 0 -0.015" rpy="0 0 0"/>
           <geometry>
              <cylinder radius="${wheel_radius}" length="${wheel_width}"/>
@@ -78,7 +80,5 @@
         <mesh filename="package://proyecto/meshes/base_link.STL"/>
       </geometry>
-      <material name="">
-        <color rgba="0.996078431372549 0.996078431372549 1 1"/>
-      </material>
+      <material name="yellow" />
     </visual>
     <collision>
@@ -86,4 +86,5 @@
       <geometry>
               <mesh filename="package://proyecto/meshes/base_link.STL"/>
+             <!-- <box size="${chasis_lenght} ${chasis_width} ${chasis_height}"/> -->
       </geometry>
     </collision>

Commit message: add pan_tilt but wont work yet

File: proyecto/urdf/proyecto.urdf.xacro (robot description, xacro)
@@ -7,7 +7,4 @@
   <xacro:property name="wheel_radius" value="0.0785" />
   <xacro:property name="wheel_width" value="0.078" />
-  <xacro:property name="chasis_lenght" value="0.581"/>
-  <xacro:property name="chasis_width" value="0.529"/>
-  <xacro:property name="chasis_height" value="0.253"/>
   <xacro:property name="pi" value="3.14159265358979323846" />
   <material name="dark_grey"><color rgba="0.2 0.2 0.2 1.0" /></material>
@@ -34,5 +31,4 @@
           <geometry>
              <cylinder radius="${wheel_radius}" length="${wheel_width}"/>
-            <!-- <mesh filename="package://proyecto/meshes/rueda_1.STL"/>-->
           </geometry>
       </collision>
@@ -86,5 +82,4 @@
       <geometry>
               <mesh filename="package://proyecto/meshes/base_link.STL"/>
-             <!-- <box size="${chasis_lenght} ${chasis_width} ${chasis_height}"/> -->
       </geometry>
     </collision>
