Commit message: ya funciona pantilt.launch pero hay que mejorar la posicion de pantilt, cambiar modelo 3d de la camara y hacer funcionar los mapas 3d

File: pckg/urdf/wxxms.xacro (robot description, xacro)
@@ -4,6 +4,4 @@
 <xacro:include filename="$(find pckg)/urdf/materials.xacro" />
 <xacro:include filename="$(find pckg)/urdf/oakd.gazebo" />
-<xacro:include filename="$(find proyecto)/urdf/proyecto.urdf.xacro">
-</xacro:include>
     <xacro:property name="flag_color" value="1"/>
     <xacro:property name="flag_depth" value="0"/>
@@ -13,5 +11,4 @@
 	<xacro:property name="oakd_cam_right_offset" value="-0.0375"/>
     <xacro:property name="real" value="$(arg is_real)" />
-<xacro:if value="$(arg use_world_frame)">
     <!--<link name="world"/>-->
     <joint name="fixed" type="fixed">
@@ -20,5 +17,4 @@
       <child link="base_linkT"/>
     </joint>
-</xacro:if>
 <link name="base_linkT">
   <inertial>
@@ -298,4 +294,89 @@
 		</sensor>
 	</xacro:if>
+        <plugin name="gazebo_ros_control" filename="libgazebo_ros_control.so">
+    </plugin>
 	</gazebo>
+  <xacro:property name="wheel_x" value="0.206" />
+  <xacro:property name="front_wheel_y" value="-0.13662" />
+  <xacro:property name="back_wheel_y" value="0.40485" />
+  <xacro:property name="wheel_z" value="-0.041" />
+  <xacro:property name="wheel_radius" value="0.0785" />
+  <xacro:property name="wheel_width" value="0.078" />
+  <xacro:property name="pi" value="3.14159265358979323846" />
+  <material name="dark_grey"><color rgba="0.2 0.2 0.2 1.0" /></material>
+  <material name="light_grey"><color rgba="0.4 0.4 0.4 1.0" /></material>
+  <material name="yellow"><color rgba="0.8 0.8 0.0 1.0" /></material>
+  <material name="black"><color rgba="0.15 0.15 0.15 1.0" /></material>
+  <xacro:macro name="wheel" params="suffix *joint_pose">
+    <link name="rueda_${suffix}">
+        <inertial>
+          <origin xyz="-5.707782267661E-07 1.62246123321108E-07 -0.0158002809636204" rpy="0 0 0"/>
+          <mass value="1.1617081622077"/>
+          <inertia ixx="0.00236389228715147" ixy="4.31489359287888E-09" ixz="-1.0352494720813E-08"
+                  iyy="0.00236389275249923" iyz="-3.84382849696802E-10" izz="0.00380474886030968"/>
+        </inertial>
+      <visual>
+        <origin xyz="0 0 0" rpy="0 0 0"/>
+          <geometry>
+            <mesh filename="package://proyecto/meshes/rueda_1.STL"/>
+          </geometry>
+          <material name="black" />
+      </visual>
+      <collision>
+        <origin xyz="0 0 -0.015" rpy="0 0 0"/>
+          <geometry>
+             <cylinder radius="${wheel_radius}" length="${wheel_width}"/>
+          </geometry>
+      </collision>
+    </link>
+    <joint name="motor_${suffix}" type="continuous">
+      <parent link="base_link"/>
+      <child link="rueda_${suffix}"/>
+      <xacro:insert_block name="joint_pose" />
+      <axis xyz="0 0 1"/>
+    </joint>
+    <transmission name="tran_${suffix}">
+      <type>transmission_interface/SimpleTransmission</type>
+      <joint name="motor_${suffix}">
+        <hardwareInterface>hardware_interface/VelocityJointInterface</hardwareInterface>
+      </joint>
+      <actuator name="actuator_${suffix}">
+        <hardwareInterface>hardware_interface/VelocityJointInterface</hardwareInterface>
+        <mechanicalReduction>1</mechanicalReduction>
+      </actuator>
+    </transmission>
+  </xacro:macro>
+  <xacro:wheel suffix="1">
+    <origin xyz="${-wheel_x} ${front_wheel_y} ${wheel_z}" rpy="${pi/2} 0 0" />
+  </xacro:wheel>
+  <xacro:wheel suffix="2">
+    <origin xyz="${wheel_x} ${front_wheel_y} ${wheel_z}" rpy="${pi/2} 0 0" />
+  </xacro:wheel>
+  <xacro:wheel suffix="3">
+    <origin xyz="${wheel_x} ${back_wheel_y} ${wheel_z}" rpy="${pi/2} 0 0" />
+  </xacro:wheel>
+  <xacro:wheel suffix="4">
+    <origin xyz="${-wheel_x} ${back_wheel_y} ${wheel_z}" rpy="${pi/2} 0 0" />
+  </xacro:wheel>
+  <link name="base_link">
+    <inertial>
+      <origin xyz="0.0238551640441538 0.0295955080939407 -0.150383488449588" rpy="0 0 0"/>
+      <mass value="4.58423641056187"/>
+      <inertia ixx="0.0171426025781744" ixy="-0.00117297644050985" ixz="-6.44110873168587E-07"
+               iyy="0.0611975209416774" iyz="-1.44180477906026E-08" izz="0.047936942239142"/>
+    </inertial>
+    <visual>
+      <origin xyz="0 0 0" rpy="0 0 0"/>
+      <geometry>
+        <mesh filename="package://proyecto/meshes/base_link.STL"/>
+      </geometry>
+      <material name="yellow" />
+    </visual>
+    <collision>
+      <origin xyz="0 0 0" rpy="0 0 0"/>
+      <geometry>
+              <mesh filename="package://proyecto/meshes/base_link.STL"/>
+      </geometry>
+    </collision>
+  </link>
 </robot>

Commit message: agregado sensor lidar y primeros pasos de navegacion, los mapas sesgiuen generando mal revisar

File: pckg/urdf/wxxms.xacro (robot description, xacro)
@@ -4,4 +4,8 @@
 <xacro:include filename="$(find pckg)/urdf/materials.xacro" />
 <xacro:include filename="$(find pckg)/urdf/oakd.gazebo" />
+  <xacro:include filename="$(find sick_tim)/urdf/sick_tim.urdf.xacro" />
+  <xacro:include filename="$(find lms1xx)/urdf/sick_lms1xx.urdf.xacro" />
+  <xacro:include filename="$(find jackal_description)/urdf/accessories/sick_lms1xx_inverted_mount.urdf.xacro" />
+  <xacro:include filename="$(find jackal_description)/urdf/accessories/sick_lms1xx_upright_mount.urdf.xacro" />
     <xacro:property name="flag_color" value="1"/>
     <xacro:property name="flag_depth" value="0"/>
@@ -172,4 +176,19 @@
 	</joint>
 	<link name="${name}_right_optical_frame"/>
+	<!--<xacro:sick_lms1xx_upright_mount topic="/laser" prefix="" parent_link="base_link">
+            <origin xyz="$(optenv JACKAL_LASER_OFFSET 0 0 0)" rpy="$(optenv JACKAL_LASER_RPY 0 0 0)" />
+          </xacro:sick_lms1xx_upright_mount> -->
+<xacro:sick_lms1xx frame="laser" topic="front/scan" />
+        <link name="front_laser"/>
+        <joint name="laser_base_joint" type="fixed">
+          <origin xyz="0 0 0.2" rpy="0 0 0"/>
+          <parent link="base_link"/>
+          <child link="front_laser"/>
+        </joint>
+        <joint name="laser_joint" type="fixed">
+          <origin xyz="0 0 0.116" rpy="0 0 0"/>
+          <parent link="front_laser"/>
+          <child link="laser"/>
+        </joint>
 	<gazebo reference="${name}_color_frame">
 	<xacro:if value="${flag_color}" >
@@ -308,4 +327,33 @@
   <material name="yellow"><color rgba="0.8 0.8 0.0 1.0" /></material>
   <material name="black"><color rgba="0.15 0.15 0.15 1.0" /></material>
+ <gazebo>
+    <plugin name="imu_controller" filename="libhector_gazebo_ros_imu.so">
+      <robotNamespace>/</robotNamespace>
+      <updateRate>50.0</updateRate>
+      <bodyName>imu_link</bodyName>
+      <topicName>imu/data</topicName>
+      <accelDrift>0.005 0.005 0.005</accelDrift>
+      <accelGaussianNoise>0.005 0.005 0.005</accelGaussianNoise>
+      <rateDrift>0.005 0.005 0.005 </rateDrift>
+      <rateGaussianNoise>0.005 0.005 0.005 </rateGaussianNoise>
+      <headingDrift>0.005</headingDrift>
+      <headingGaussianNoise>0.005</headingGaussianNoise>
+    </plugin>
+  </gazebo>
+  <gazebo>
+    <plugin name="gps_controller" filename="libhector_gazebo_ros_gps.so">
+      <updateRate>40</updateRate>
+      <robotNamespace>/</robotNamespace>
+      <bodyName>navsat_link</bodyName>
+      <frameId>base_link</frameId>
+      <topicName>/navsat/fix</topicName>
+      <velocityTopicName>/navsat/vel</velocityTopicName>
+      <referenceLatitude>$(optenv GAZEBO_WORLD_LAT 49.9)</referenceLatitude>
+      <referenceLongitude>$(optenv GAZEBO_WORLD_LON 8.9)</referenceLongitude>
+      <referenceHeading>90</referenceHeading>
+      <referenceAltitude>0</referenceAltitude>
+      <drift>0.0001 0.0001 0.0001</drift>
+    </plugin>
+  </gazebo>
   <xacro:macro name="wheel" params="suffix *joint_pose">
     <link name="rueda_${suffix}">

Commit message: ya funciona proyecto, falta de cambiar el modelo de la camara y alinear tanto el lidar como el opantilt al centro del robot

File: pckg/urdf/wxxms.xacro (robot description, xacro)
@@ -17,5 +17,5 @@
     <!--<link name="world"/>-->
     <joint name="fixed" type="fixed">
-        <origin xyz="0 0 0.5" rpy="0 0 0" />
+        <origin xyz="0.2 0.2 0.15" rpy="0 0 0" />
       <parent link="base_link"/>
       <child link="base_linkT"/>
@@ -382,5 +382,5 @@
       <child link="rueda_${suffix}"/>
       <xacro:insert_block name="joint_pose" />
-      <axis xyz="0 0 1"/>
+      <axis xyz="0 0 -1"/>
     </joint>
     <transmission name="tran_${suffix}">

Commit message: comentar parte imu_controller y alinear laser con pan_tilt

File: pckg/urdf/wxxms.xacro (robot description, xacro)
@@ -17,5 +17,5 @@
     <!--<link name="world"/>-->
     <joint name="fixed" type="fixed">
-        <origin xyz="0.2 0.2 0.15" rpy="0 0 0" />
+        <origin xyz="0.126 0.15 0.17" rpy="0 0 1.570796327" />
       <parent link="base_link"/>
       <child link="base_linkT"/>
@@ -30,5 +30,5 @@
     <origin xyz="0 0 0" rpy="0 0 0"/>
     <geometry>
-      <mesh filename="package://pckg/meshes/base_link.stl" scale="0.001 0.001 0.001"/>
+      <mesh filename="package://pckg/meshes/base_link2.stl" scale="0.001 0.001 0.001"/>
     </geometry>
     <material name="silver"/>
@@ -37,5 +37,5 @@
     <origin xyz="0 0 0" rpy="0 0 0"/>
     <geometry>
-      <mesh filename="package://pckg/meshes/base_link.stl" scale="0.001 0.001 0.001"/>
+      <mesh filename="package://pckg/meshes/base_link2.stl" scale="0.001 0.001 0.001"/>
     </geometry>
   </collision>
@@ -182,5 +182,5 @@
         <link name="front_laser"/>
         <joint name="laser_base_joint" type="fixed">
-          <origin xyz="0 0 0.2" rpy="0 0 0"/>
+          <origin xyz="0 0.15 0.17" rpy="0 0 0"/>
           <parent link="base_link"/>
           <child link="front_laser"/>
@@ -327,4 +327,5 @@
   <material name="yellow"><color rgba="0.8 0.8 0.0 1.0" /></material>
   <material name="black"><color rgba="0.15 0.15 0.15 1.0" /></material>
+<!--
  <gazebo>
     <plugin name="imu_controller" filename="libhector_gazebo_ros_imu.so">
@@ -356,4 +357,5 @@
     </plugin>
   </gazebo>
+-->
   <xacro:macro name="wheel" params="suffix *joint_pose">
     <link name="rueda_${suffix}">
